Commit message: rviz works

File: src/ulixarm_description/urdf/ulixarm.urdf (robot description, URDF)
Before this commit: robot ulixarm, 8 links, 7 joints
Links:
- link base_link: geometry collision mesh filename=package://ulixarm_description/meshes/collision/base.stl; visual mesh filename=package://ulixarm_description/meshes/visual/base.stl
- link link1: geometry collision mesh filename=package://ulixarm_description/meshes/collision/joint1.stl; visual mesh filename=package://ulixarm_description/meshes/visual/joint1.stl
- link link2: geometry collision mesh filename=package://ulixarm_description/meshes/collision/link1.stl; visual mesh filename=package://ulixarm_description/meshes/visual/link1.stl
- link link3: geometry collision mesh filename=package://ulixarm_description/meshes/collision/link2.stl; visual mesh filename=package://ulixarm_description/meshes/visual/link2.stl
- link link4: geometry collision mesh filename=package://ulixarm_description/meshes/collision/joint4.stl; visual mesh filename=package://ulixarm_description/meshes/visual/joint4.stl
- link link5: geometry collision mesh filename=package://ulixarm_description/meshes/collision/joint5.stl; visual mesh filename=package://ulixarm_description/meshes/visual/joint5.stl
Joints:
- joint joint1: limit lower=-3.15 upper=3.15 effort=0.5 velocity=0.10 -> lower=-1.57079632679 upper=1.57079632679 effort=0.5 velocity=0.10
- joint joint2: limit lower=-3.15 upper=3.15 effort=0.5 velocity=0.10 -> lower=-1.57079632679 upper=1.57079632679 effort=0.5 velocity=0.10
- joint joint3: limit lower=-3.15 upper=3.15 effort=0.5 velocity=0.10 -> lower=-1.57079632679 upper=2.7925268 effort=0.5 velocity=0.10
- joint joint4: limit lower=-3.15 upper=3.15 effort=0.5 velocity=0.10 -> lower=-3.14159265359 upper=1.57079632679 effort=0.5 velocity=0.10
- joint joint5: limit lower=-3.15 upper=3.15 effort=0.5 velocity=0.10 -> lower=-1.57079632679 upper=1.57079632679 effort=0.5 velocity=0.10
- joint joint6: limit lower=-3.15 upper=3.15 effort=0.5 velocity=0.10 -> lower=-1.57079632679 upper=1.57079632679 effort=0.5 velocity=0.10

Commit message: edit joint5 axis direction

File: src/ulixarm_description/urdf/ulixarm.urdf (robot description, URDF)
Before this commit: robot ulixarm, 8 links, 7 joints
Joints:
- joint joint5: axis 0 0 1 -> 0 0 -1

Commit message: added xacro

File: src/ulixarm_description/urdf/ulixarm.urdf (robot description, URDF)
Before this commit: robot ulixarm, 8 links, 7 joints
Links:
- removed link base_link
- added link base, mass 1.0; collision mesh filename=package://ulixarm_description/meshes/collision/base.stl; visual mesh filename=package://ulixarm_description/meshes/visual/base.stl
- link link1: mass None -> 1.0
- link link2: mass None -> 1.0
- link link3: mass None -> 1.0
- link link4: mass None -> 1.0
- link link5: mass None -> 1.0
Joints:
- joint joint0: child base_link -> base
- joint joint1: limit lower=-1.57079632679 upper=1.57079632679 effort=0.5 velocity=0.10 -> lower=${-PI/2} upper=${PI/2} effort=${effort_limit_DM4340} velocity=${velocity_limit_DM4340}; parent base_link -> base
- joint joint2: limit lower=-1.57079632679 upper=1.57079632679 effort=0.5 velocity=0.10 -> lower=${-PI/2} upper=${PI/2} effort=${effort_limit_DM4340} velocity=${velocity_limit_DM4340}; origin xyz=0.027175 0. 0.0425 rpy=3.14159265359 -1.57079632679 0. -> xyz=0.027175 0. 0.0425 rpy=${PI} ${-PI/2} 0.
- joint joint3: limit lower=-1.57079632679 upper=2.7925268 effort=0.5 velocity=0.10 -> lower=${-PI/2} upper=2.7925268 effort=${effort_limit_DM4340} velocity=${velocity_limit_DM4340}; origin xyz=0.280 0. -0.0473 rpy=3.14159265359 0. 0. -> xyz=0.280 0. -0.0473 rpy=${PI} 0. 0.
- joint joint4: limit lower=-3.14159265359 upper=1.57079632679 effort=0.5 velocity=0.10 -> lower=${-PI} upper=${PI/2} effort=${effort_limit_DM4310} velocity=${velocity_limit_DM4310}; origin xyz=0.260 0. -0.040 rpy=3.14159265359 0. -1.57079632679 -> xyz=0.260 0. -0.040 rpy=${PI} 0. ${-PI/2}
- joint joint5: limit lower=-1.57079632679 upper=1.57079632679 effort=0.5 velocity=0.10 -> lower=${-PI/2} upper=${PI/2} effort=${effort_limit_DM4310} velocity=${velocity_limit_DM4310}; origin xyz=0.046 0. 0.031 rpy=1.57079632679 0. -1.57079632679 -> xyz=0.046 0. 0.031 rpy=${PI/2} 0. ${-PI/2}
- joint joint6: limit lower=-1.57079632679 upper=1.57079632679 effort=0.5 velocity=0.10 -> lower=${-PI/2} upper=${PI/2} effort=${effort_limit_DM4310} velocity=${velocity_limit_DM4310}; origin xyz=0.0825 0. -0.0235 rpy=1.57079632679 0. 1.57079632679 -> xyz=0.0825 0. -0.0235 rpy=${PI/2} 0. ${PI/2}

Commit message: added moveit config

File: src/ulixarm_description/urdf/ulixarm.urdf (robot description, URDF)
Before this commit: robot ulixarm, 8 links, 7 joints
Links:
- removed link world
- link base: mass 1.0 -> None
Joints:
- removed joint joint0

File: src/ulixarm_description/urdf/ulixarm.urdf.xacro (robot description, xacro)
@@ -1,5 +1,5 @@
 <?xml version="1.0" ?>
 <!-- =================================================================================== -->
-<!-- |    This document was autogenerated by xacro from src/ulixarm_description/urdf/ulixarm.urdf | -->
+<!-- |    This document was autogenerated by xacro from ulixarm_description/urdf/ulixarm.urdf | -->
 <!-- |    EDITING THIS FILE BY HAND IS NOT RECOMMENDED                                 | -->
 <!-- =================================================================================== -->
@@ -8,5 +8,4 @@
   <!-- CONSTANTS -->
   <!-- LINKS -->
-  <link name="world"/>
   <link name="base">
     <visual>
@@ -22,8 +21,4 @@
       </geometry>
     </collision>
-    <inertial>
-      <mass value="1.0"/>
-      <inertia ixx="1.0" ixy="0.0" ixz="0.0" iyy="1.0" iyz="0.0" izz="1.0"/>
-    </inertial>
   </link>
   <link name="link1">
@@ -119,10 +114,4 @@
   <link name="tcp"/>
   <!-- JOINTS -->
-  <joint name="joint0" type="fixed">
-    <origin rpy="0. 0. 0." xyz="0. 0. 0."/>
-    <parent link="world"/>
-    <child link="base"/>
-    <limit effort="0.0" lower="0.0" upper="0.0" velocity="0.0"/>
-  </joint>
   <joint name="joint1" type="revolute">
     <origin rpy="0. 0. 0." xyz="0. 0. 0.0533"/>

File: src/ulixarm_moveit_config/config/ulixarm.ros2_control.xacro (robot description, xacro)
@@ -10,5 +10,4 @@
             <joint name="joint1">
                 <command_interface name="position"/>
-                <command_interface name="velocity"/>
                 <state_interface name="position">
                   <param name="initial_value">${initial_positions['joint1']}</param>
@@ -18,5 +17,4 @@
             <joint name="joint2">
                 <command_interface name="position"/>
-                <command_interface name="velocity"/>
                 <state_interface name="position">
                   <param name="initial_value">${initial_positions['joint2']}</param>
@@ -26,5 +24,4 @@
             <joint name="joint3">
                 <command_interface name="position"/>
-                <command_interface name="velocity"/>
                 <state_interface name="position">
                   <param name="initial_value">${initial_positions['joint3']}</param>
@@ -34,5 +31,4 @@
             <joint name="joint4">
                 <command_interface name="position"/>
-                <command_interface name="velocity"/>
                 <state_interface name="position">
                   <param name="initial_value">${initial_positions['joint4']}</param>
@@ -42,5 +38,4 @@
             <joint name="joint5">
                 <command_interface name="position"/>
-                <command_interface name="velocity"/>
                 <state_interface name="position">
                   <param name="initial_value">${initial_positions['joint5']}</param>
@@ -50,5 +45,4 @@
             <joint name="joint6">
                 <command_interface name="position"/>
-                <command_interface name="velocity"/>
                 <state_interface name="position">
                   <param name="initial_value">${initial_positions['joint6']}</param>

File: src/ulixarm_moveit_config/config/ulixarm.urdf.xacro (robot description, xacro)
@@ -3,5 +3,5 @@
     <xacro:arg name="initial_positions_file" default="initial_positions.yaml" />
     <!-- Import ulixarm urdf file -->
-    <xacro:include filename="$(find ulixarm_description)/urdf/ulixarm.urdf" />
+    <xacro:include filename="$(find ulixarm_description)/urdf/ulixarm.urdf.xacro" />
     <!-- Import control_xacro -->
     <xacro:include filename="ulixarm.ros2_control.xacro" />
