Commit message: added ulixhand description

File: src/ulixarm_description/urdf/ulixarm.urdf.xacro (robot description, xacro)
@@ -1,158 +1,159 @@
-<?xml version="1.0" ?>
-<!-- =================================================================================== -->
-<!-- |    This document was autogenerated by xacro from ulixarm_description/urdf/ulixarm.urdf | -->
-<!-- |    EDITING THIS FILE BY HAND IS NOT RECOMMENDED                                 | -->
-<!-- =================================================================================== -->
-<robot name="ulixarm">
-  <!-- run: xacro ulixarm.urdf > ulixarm.xacro -->
-  <!-- CONSTANTS -->
-  <!-- LINKS -->
-  <link name="base">
-    <visual>
-      <origin xyz="0. 0. 0."/>
-      <geometry>
-        <mesh filename="package://ulixarm_description/meshes/visual/base.stl"/>
-      </geometry>
-    </visual>
-    <collision>
-      <origin xyz="0. 0. 0."/>
-      <geometry>
-        <mesh filename="package://ulixarm_description/meshes/collision/base.stl"/>
-      </geometry>
-    </collision>
-  </link>
-  <link name="link1">
-    <visual>
-      <origin xyz="0. 0. 0."/>
-      <geometry>
-        <mesh filename="package://ulixarm_description/meshes/visual/joint1.stl"/>
-      </geometry>
-    </visual>
-    <collision>
-      <origin xyz="0. 0. 0."/>
-      <geometry>
-        <mesh filename="package://ulixarm_description/meshes/collision/joint1.stl"/>
-      </geometry>
-    </collision>
-    <inertial>
-      <mass value="1.0"/>
-      <inertia ixx="1.0" ixy="0.0" ixz="0.0" iyy="1.0" iyz="0.0" izz="1.0"/>
-    </inertial>
-  </link>
-  <link name="link2">
-    <visual>
-      <origin xyz="0. 0. 0."/>
-      <geometry>
-        <mesh filename="package://ulixarm_description/meshes/visual/link1.stl"/>
-      </geometry>
-    </visual>
-    <collision>
-      <origin xyz="0. 0. 0."/>
-      <geometry>
-        <mesh filename="package://ulixarm_description/meshes/collision/link1.stl"/>
-      </geometry>
-    </collision>
-    <inertial>
-      <mass value="1.0"/>
-      <inertia ixx="1.0" ixy="0.0" ixz="0.0" iyy="1.0" iyz="0.0" izz="1.0"/>
-    </inertial>
-  </link>
-  <link name="link3">
-    <visual>
-      <origin xyz="0. 0. 0."/>
-      <geometry>
-        <mesh filename="package://ulixarm_description/meshes/visual/link2.stl"/>
-      </geometry>
-    </visual>
-    <collision>
-      <origin xyz="0. 0. 0."/>
-      <geometry>
-        <mesh filename="package://ulixarm_description/meshes/collision/link2.stl"/>
-      </geometry>
-    </collision>
-    <inertial>
-      <mass value="1.0"/>
-      <inertia ixx="1.0" ixy="0.0" ixz="0.0" iyy="1.0" iyz="0.0" izz="1.0"/>
-    </inertial>
-  </link>
-  <link name="link4">
-    <visual>
-      <origin xyz="0. 0. 0."/>
-      <geometry>
-        <mesh filename="package://ulixarm_description/meshes/visual/joint4.stl"/>
-      </geometry>
-    </visual>
-    <collision>
-      <origin xyz="0. 0. 0."/>
-      <geometry>
-        <mesh filename="package://ulixarm_description/meshes/collision/joint4.stl"/>
-      </geometry>
-    </collision>
-    <inertial>
-      <mass value="1.0"/>
-      <inertia ixx="1.0" ixy="0.0" ixz="0.0" iyy="1.0" iyz="0.0" izz="1.0"/>
-    </inertial>
-  </link>
-  <link name="link5">
-    <visual>
-      <origin xyz="0. 0. 0."/>
-      <geometry>
-        <mesh filename="package://ulixarm_description/meshes/visual/joint5.stl"/>
-      </geometry>
-    </visual>
-    <collision>
-      <origin xyz="0. 0. 0."/>
-      <geometry>
-        <mesh filename="package://ulixarm_description/meshes/collision/joint5.stl"/>
-      </geometry>
-    </collision>
-    <inertial>
-      <mass value="1.0"/>
-      <inertia ixx="1.0" ixy="0.0" ixz="0.0" iyy="1.0" iyz="0.0" izz="1.0"/>
-    </inertial>
-  </link>
-  <link name="tcp"/>
-  <!-- JOINTS -->
-  <joint name="joint1" type="revolute">
-    <origin rpy="0. 0. 0." xyz="0. 0. 0.0533"/>
-    <parent link="base"/>
-    <child link="link1"/>
-    <axis xyz="0 0 1"/>
-    <limit effort="27.0" lower="-1.570796326795" upper="1.570796326795" velocity="8.0"/>
-  </joint>
-  <joint name="joint2" type="revolute">
-    <origin rpy="3.14159265359 -1.570796326795 0." xyz="0.027175 0. 0.0425"/>
-    <parent link="link1"/>
-    <child link="link2"/>
-    <axis xyz="0 0 1"/>
-    <limit effort="27.0" lower="-1.570796326795" upper="1.570796326795" velocity="8.0"/>
-  </joint>
-  <joint name="joint3" type="revolute">
-    <origin rpy="3.14159265359 0. 0." xyz="0.280 0. -0.0473"/>
-    <parent link="link2"/>
-    <child link="link3"/>
-    <axis xyz="0 0 1"/>
-    <limit effort="27.0" lower="-1.570796326795" upper="2.7925268" velocity="8.0"/>
-  </joint>
-  <joint name="joint4" type="revolute">
-    <origin rpy="3.14159265359 0. -1.570796326795" xyz="0.260 0. -0.040"/>
-    <parent link="link3"/>
-    <child link="link4"/>
-    <axis xyz="0 0 1"/>
-    <limit effort="10.0" lower="-3.14159265359" upper="1.570796326795" velocity="30.0"/>
-  </joint>
-  <joint name="joint5" type="revolute">
-    <origin rpy="1.570796326795 0. -1.570796326795" xyz="0.046 0. 0.031"/>
-    <parent link="link4"/>
-    <child link="link5"/>
-    <axis xyz="0 0 -1"/>
-    <limit effort="10.0" lower="-1.570796326795" upper="1.570796326795" velocity="30.0"/>
-  </joint>
-  <joint name="joint6" type="revolute">
-    <origin rpy="1.570796326795 0. 1.570796326795" xyz="0.0825 0. -0.0235"/>
-    <parent link="link5"/>
-    <child link="tcp"/>
-    <axis xyz="0 0 1"/>
-    <limit effort="10.0" lower="-1.570796326795" upper="1.570796326795" velocity="30.0"/>
-  </joint>
+<?xml version="1.0"?>
+<robot xmlns:xacro="http://www.ros.org/wiki/xacro" name="ulixarm">
+    <!-- run: xacro ulixarm.urdf > ulixarm.xacro -->
+    <!-- CONSTANTS -->
+    <xacro:property name="PI" value="3.14159265359"/>
+    <xacro:property name="velocity_limit_DM4340"   value="8.0"/>
+    <xacro:property name="effort_limit_DM4340"  value="27.0"/>
+    <xacro:property name="velocity_limit_DM4310"   value="30.0"/>
+    <xacro:property name="effort_limit_DM4310"  value="10.0"/>
+    <!-- LINKS -->
+    <link name="base_link">
+        <visual>
+            <origin xyz="0. 0. 0."/>
+            <geometry>
+                <mesh filename="package://ulixarm_description/meshes/visual/base.stl"/>
+            </geometry>
+        </visual>
+        <collision>
+            <origin xyz="0. 0. 0."/>
+            <geometry>
+                <mesh filename="package://ulixarm_description/meshes/collision/base.stl"/>
+            </geometry>
+        </collision>
+    </link>
+    <link name="link1">
+        <visual>
+            <origin xyz="0. 0. 0."/>
+            <geometry>
+                <mesh filename="package://ulixarm_description/meshes/visual/joint1.stl"/>
+            </geometry>
+        </visual>
+        <collision>
+            <origin xyz="0. 0. 0."/>
+            <geometry>
+                <mesh filename="package://ulixarm_description/meshes/collision/joint1.stl"/>
+            </geometry>
+        </collision>
+        <inertial>
+            <mass value="1.0"/>
+            <inertia ixx="1.0" ixy="0.0" ixz="0.0" iyy="1.0" iyz="0.0" izz="1.0"/>
+        </inertial>
+    </link>
+    <link name="link2">
+        <visual>
+            <origin xyz="0. 0. 0."/>
+            <geometry>
+                <mesh filename="package://ulixarm_description/meshes/visual/link1.stl"/>
+            </geometry>
+        </visual>
+        <collision>
+            <origin xyz="0. 0. 0."/>
+            <geometry>
+                <mesh filename="package://ulixarm_description/meshes/collision/link1.stl"/>
+            </geometry>
+        </collision>
+        <inertial>
+            <mass value="1.0"/>
+            <inertia ixx="1.0" ixy="0.0" ixz="0.0" iyy="1.0" iyz="0.0" izz="1.0"/>
+        </inertial>
+    </link>
+    <link name="link3">
+        <visual>
+            <origin xyz="0. 0. 0."/>
+            <geometry>
+                <mesh filename="package://ulixarm_description/meshes/visual/link2.stl"/>
+            </geometry>
+        </visual>
+        <collision>
+            <origin xyz="0. 0. 0."/>
+            <geometry>
+                <mesh filename="package://ulixarm_description/meshes/collision/link2.stl"/>
+            </geometry>
+        </collision>
+        <inertial>
+            <mass value="1.0"/>
+            <inertia ixx="1.0" ixy="0.0" ixz="0.0" iyy="1.0" iyz="0.0" izz="1.0"/>
+        </inertial>
+    </link>
+    <link name="link4">
+        <visual>
+            <origin xyz="0. 0. 0."/>
+            <geometry>
+                <mesh filename="package://ulixarm_description/meshes/visual/joint4.stl"/>
+            </geometry>
+        </visual>
+        <collision>
+            <origin xyz="0. 0. 0."/>
+            <geometry>
+                <mesh filename="package://ulixarm_description/meshes/collision/joint4.stl"/>
+            </geometry>
+        </collision>
+        <inertial>
+            <mass value="1.0"/>
+            <inertia ixx="1.0" ixy="0.0" ixz="0.0" iyy="1.0" iyz="0.0" izz="1.0"/>
+        </inertial>
+    </link>
+    <link name="link5">
+        <visual>
+            <origin xyz="0. 0. 0."/>
+            <geometry>
+                <mesh filename="package://ulixarm_description/meshes/visual/joint5.stl"/>
+            </geometry>
+        </visual>
+        <collision>
+            <origin xyz="0. 0. 0."/>
+            <geometry>
+                <mesh filename="package://ulixarm_description/meshes/collision/joint5.stl"/>
+            </geometry>
+        </collision>
+        <inertial>
+            <mass value="1.0"/>
+            <inertia ixx="1.0" ixy="0.0" ixz="0.0" iyy="1.0" iyz="0.0" izz="1.0"/>
+        </inertial>
+    </link>
+    <link name="tool0"></link>
+    <!-- JOINTS -->
+    <joint name="joint1" type="revolute">
+        <origin xyz="0. 0. 0.0533" rpy="0. 0. 0."/>
+        <parent link="base_link"/>
+        <child link="link1"/>
+        <axis xyz="0 0 1"/>
+        <limit lower="${-PI/2}" upper="${PI/2}" velocity="${velocity_limit_DM4340}" effort="${effort_limit_DM4340}"/>
+    </joint>
+    <joint name="joint2" type="revolute">
+        <origin xyz="0.027175 0. 0.0425" rpy="${PI} ${-PI/2} 0."/>
+        <parent link="link1"/>
+        <child link="link2"/>
+        <axis xyz="0 0 1"/>
+        <limit lower="${-PI/2}" upper="${PI/2}" velocity="${velocity_limit_DM4340}" effort="${effort_limit_DM4340}"/>
+    </joint>
+    <joint name="joint3" type="revolute">
+        <origin xyz="0.280 0. -0.0473" rpy="${PI} 0. 0."/>
+        <parent link="link2"/>
+        <child link="link3"/>
+        <axis xyz="0 0 1"/>
+        <limit lower="${-PI/2}" upper="2.7925268" velocity="${velocity_limit_DM4340}" effort="${effort_limit_DM4340}"/>
+    </joint>
+    <joint name="joint4" type="revolute">
+        <origin xyz="0.260 0. -0.040" rpy="${PI} 0. ${-PI/2}"/>
+        <parent link="link3"/>
+        <child link="link4"/>
+        <axis xyz="0 0 1"/>
+        <limit lower="${-PI}" upper="${PI/2}" velocity="${velocity_limit_DM4310}" effort="${effort_limit_DM4310}"/>
+    </joint>
+    <joint name="joint5" type="revolute">
+        <origin xyz="0.046 0. 0.031" rpy="${PI/2} 0. ${-PI/2}"/>
+        <parent link="link4"/>
+        <child link="link5"/>
+        <axis xyz="0 0 -1"/>
+        <limit lower="${-PI/2}" upper="${PI/2}" velocity="${velocity_limit_DM4310}" effort="${effort_limit_DM4310}"/>
+    </joint>
+    <joint name="joint6" type="revolute">
+        <origin xyz="0.0825 0. -0.0235" rpy="${PI/2} 0. ${PI/2}"/>
+        <parent link="link5"/>
+        <child link="tool0"/>
+        <axis xyz="0 0 1"/>
+        <limit lower="${-PI/2}" upper="${PI/2}" velocity="${velocity_limit_DM4310}" effort="${effort_limit_DM4310}"/>
+    </joint>
 </robot>
