Commit message: added gripper

File: src/ulixarm_description/urdf/robot.urdf.xacro (robot description, xacro)
@@ -1,15 +1,15 @@
 <?xml version="1.0"?>
-<robot xmlns:xacro="http://www.ros.org/wiki/xacro" name="ulixarm_with_ulixhand">
-  <!-- Include both xacro files -->
-  <xacro:include filename="$(find ulixarm_description)/urdf/ulixarm.urdf.xacro"/>
-  <xacro:include filename="$(find ulixarm_description)/urdf/ulixhand.urdf.xacro"/>
-  <!-- Instantiate the arm (defines base_link → tool0) -->
-  <xacro:arm_macro prefix="arm_"/>
-  <!-- Instantiate the gripper, parented to the arm's tool flange -->
-  <xacro:gripper_macro prefix="hand_"/>
+<robot xmlns:xacro="http://www.ros.org/wiki/xacro" name="ulixarm">
+  <xacro:property name="MANIPULATOR_PREFIX" value="manipulator_"/>
+  <xacro:property name="GRIPPER_PREFIX" value="gripper_"/>
+  <!-- Include xacro files -->
+  <xacro:include filename="$(find ulixarm_description)/urdf/manipulator.urdf.xacro"/>
+  <xacro:include filename="$(find ulixarm_description)/urdf/gripper.urdf.xacro"/>
+  <xacro:manipulator_macro prefix="${MANIPULATOR_PREFIX}"/>
+  <xacro:gripper_macro prefix="${GRIPPER_PREFIX}"/>
   <!-- Attach gripper base to the arm's end-effector link -->
-  <joint name="ulixarm_to_ulixhand" type="fixed">
-    <parent link="arm_tool0"/>
-    <child  link="hand_base_link"/>
+  <joint name="manipulator_to_gripper" type="fixed">
+    <parent link="${MANIPULATOR_PREFIX}tool0"/>
+    <child  link="${GRIPPER_PREFIX}base_link"/>
     <origin xyz="0 0 0" rpy="0 0 0"/>
   </joint>

File: src/ulixarm_moveit_config/config/ulixarm.ros2_control.xacro (robot description, xacro)
@@ -8,4 +8,5 @@
                 <!-- <plugin>mock_components/GenericSystem</plugin> -->
                 <plugin>ulixarm_hardware/RobotSystem</plugin>
+                <param name="port">/dev/ttyUSB0</param>
             </hardware>
             <joint name="joint1">
@@ -57,4 +58,12 @@
                 <state_interface name="velocity"/>
             </joint>
+            <joint name="finger_right_joint">
+                <command_interface name="position"/>
+                <command_interface name="velocity"/>
+                <state_interface name="position">
+                  <param name="initial_value">${initial_positions['finger_right_joint']}</param>
+                </state_interface>
+                <state_interface name="velocity"/>
+            </joint>
         </ros2_control>
     </xacro:macro>

File: src/ulixarm_moveit_config/config/ulixarm.urdf.xacro (robot description, xacro)
@@ -3,8 +3,7 @@
     <xacro:arg name="initial_positions_file" default="initial_positions.yaml" />
     <!-- Import ulixarm urdf file -->
-    <xacro:include filename="$(find ulixarm_description)/urdf/ulixarm.urdf.xacro" />
+    <xacro:include filename="$(find ulixarm_description)/urdf/robot.urdf" />
     <!-- Import control_xacro -->
     <xacro:include filename="ulixarm.ros2_control.xacro" />
-    <!-- <xacro:ulixarm_ros2_control name="FakeSystem" initial_positions_file="$(arg initial_positions_file)"/> -->
-    <xacro:ulixarm_ros2_control name="ulixarm" initial_positions_file="$(arg initial_positions_file)"/>
+    <xacro:ulixarm_ros2_control name="FakeSystem" initial_positions_file="$(arg initial_positions_file)"/>
 </robot>
