Commit message: added textures

File: src/ulixarm_description/urdf/manipulator.urdf.xacro (robot description, xacro)
@@ -13,5 +13,5 @@
                 <origin xyz="0. 0. 0."/>
                 <geometry>
-                    <mesh filename="package://ulixarm_description/meshes/visual/base.stl"/>
+                    <mesh filename="package://ulixarm_description/meshes/visual/base_link.dae"/>
                 </geometry>
             </visual>
@@ -32,5 +32,5 @@
                 <origin xyz="0. 0. 0."/>
                 <geometry>
-                    <mesh filename="package://ulixarm_description/meshes/visual/joint1.stl"/>
+                    <mesh filename="package://ulixarm_description/meshes/visual/link1.dae"/>
                 </geometry>
             </visual>
@@ -51,5 +51,5 @@
                 <origin xyz="0. 0. 0."/>
                 <geometry>
-                    <mesh filename="package://ulixarm_description/meshes/visual/link1.stl"/>
+                    <mesh filename="package://ulixarm_description/meshes/visual/link2.dae"/>
                 </geometry>
             </visual>
@@ -70,5 +70,5 @@
                 <origin xyz="0. 0. 0."/>
                 <geometry>
-                    <mesh filename="package://ulixarm_description/meshes/visual/link2.stl"/>
+                    <mesh filename="package://ulixarm_description/meshes/visual/link3.dae"/>
                 </geometry>
             </visual>
@@ -90,5 +90,5 @@
                 <origin xyz="0. 0. 0."/>
                 <geometry>
-                    <mesh filename="package://ulixarm_description/meshes/visual/joint4.stl"/>
+                    <mesh filename="package://ulixarm_description/meshes/visual/link4.dae"/>
                 </geometry>
             </visual>
@@ -110,5 +110,5 @@
                 <origin xyz="0. 0. 0."/>
                 <geometry>
-                    <mesh filename="package://ulixarm_description/meshes/visual/joint5.stl"/>
+                    <mesh filename="package://ulixarm_description/meshes/visual/link5.dae"/>
                 </geometry>
             </visual>
