Commit message: fixed cg link 4

File: src/ulixarm_description/urdf/manipulator.urdf.xacro (robot description, xacro)
@@ -94,7 +94,7 @@
             </collision>
             <inertial>
-                <origin xyz="0.024 -0.017 0.048"/>
-                <mass value="0.072"/>
-                <inertia ixx="0.000075" ixy="0.0" ixz="0.0" iyy="0.000084" iyz="0.0" izz="0.000095"/>
+                <origin xyz="0.024 -0.017 -0.012"/>
+                <mass value="0.175"/>
+                <inertia ixx="0.000187" ixy="0.000068" ixz="0.000068" iyy="0.000206" iyz="-0.000047" izz="0.000235"/>
             </inertial>
         </link>

File: src/ulixarm_description/urdf/robot.urdf (robot description, URDF)
Before this commit: robot ulixarm, 11 links, 10 joints
Links:
- link manipulator_link4: mass 0.072 -> 0.175
