Commit message: edit finger offset

File: src/ulixarm_description/urdf/gripper.urdf.xacro (robot description, xacro)
@@ -20,4 +20,8 @@
                 </geometry>
             </collision>
+            <inertial>
+                <mass value="1.0"/>
+                <inertia ixx="1.0" ixy="0.0" ixz="0.0" iyy="1.0" iyz="0.0" izz="1.0"/>
+            </inertial>
         </link>
         <link name="${prefix}finger_right">
@@ -59,5 +63,5 @@
         <!-- JOINTS -->
         <joint name="finger_right_joint" type="prismatic">
-            <origin xyz="0. 0. 0.1219" rpy="0. 0. 0."/>
+            <origin xyz="0. 0. 0.1349" rpy="0. 0. 0."/>
             <parent link="${prefix}base_link"/>
             <child link="${prefix}finger_right"/>
@@ -66,5 +70,5 @@
         </joint>
         <joint name="finger_left_joint" type="prismatic">
-            <origin xyz="0. 0. 0.1219" rpy="0. 0. ${PI}"/>
+            <origin xyz="0. 0. 0.1349" rpy="0. 0. ${PI}"/>
             <parent link="${prefix}base_link"/>
             <child link="${prefix}finger_left"/>

Commit message: fixed mimic joint

File: src/ulixarm_description/urdf/gripper.urdf.xacro (robot description, xacro)
@@ -67,5 +67,5 @@
             <child link="${prefix}finger_right"/>
             <axis xyz="1 0 0"/>
-            <limit lower="-0.05" upper="0.038" velocity="${velocity_limit_DMJ3507}" effort="${effort_limit_DMJ3507}"/>
+            <limit lower="0.0" upper="0.038" velocity="${velocity_limit_DMJ3507}" effort="${effort_limit_DMJ3507}"/>
         </joint>
         <joint name="finger_left_joint" type="prismatic">
@@ -73,7 +73,7 @@
             <parent link="${prefix}base_link"/>
             <child link="${prefix}finger_left"/>
-            <axis xyz="-1 0 0"/>
-            <mimic joint="finger_right_joint" multiplier="-1" offset="0"/>
-            <limit lower="-0.038" upper="0.05" velocity="${velocity_limit_DMJ3507}" effort="${effort_limit_DMJ3507}"/>
+            <axis xyz="1 0 0"/>
+            <mimic joint="finger_right_joint" multiplier="1" offset="0"/>
+            <limit lower="0.0" upper="0.038" velocity="${velocity_limit_DMJ3507}" effort="${effort_limit_DMJ3507}"/>
         </joint>
   </xacro:macro>

File: src/ulixarm_description/urdf/robot.urdf (robot description, URDF)
Before this commit: robot ulixarm, 11 links, 10 joints
Links:
- link gripper_base_link: mass None -> 1.0
Joints:
- joint finger_left_joint: axis -1 0 0 -> 1 0 0; limit lower=-0.038 upper=0.05 effort=1.0 velocity=1.0 -> lower=0.0 upper=0.038 effort=0.1 velocity=0.5; mimic joint=finger_right_joint multiplier=-1 offset=0 -> joint=finger_right_joint multiplier=1 offset=0; origin xyz=0. 0. 0.1219 rpy=0. 0. 3.14159265359 -> xyz=0. 0. 0.1349 rpy=0. 0. 3.14159265359
- joint finger_right_joint: limit lower=-0.05 upper=0.038 effort=1.0 velocity=1.0 -> lower=0.0 upper=0.038 effort=0.1 velocity=0.5; origin xyz=0. 0. 0.1219 rpy=0. 0. 0. -> xyz=0. 0. 0.1349 rpy=0. 0. 0.

File: src/ulixarm_moveit_config/config/ulixarm.ros2_control.xacro (robot description, xacro)
@@ -6,6 +6,6 @@
             <hardware>
                 <!-- By default, set up controllers for simulation. This won't work on real hardware -->
-                <!-- <plugin>mock_components/GenericSystem</plugin> -->
-                <plugin>ulixarm_hardware/RobotSystem</plugin>
+                <plugin>mock_components/GenericSystem</plugin>
+                <!-- <plugin>ulixarm_hardware/RobotSystem</plugin> -->
                 <param name="port">/dev/ttyUSB0</param>
             </hardware>

Commit message: added inertial tag

File: src/ulixarm_description/urdf/gripper.urdf.xacro (robot description, xacro)
@@ -21,6 +21,7 @@
             </collision>
             <inertial>
-                <mass value="1.0"/>
-                <inertia ixx="1.0" ixy="0.0" ixz="0.0" iyy="1.0" iyz="0.0" izz="1.0"/>
+                <origin xyz="0. 0. 0.052"/>
+                <mass value="0.489"/>
+                <inertia ixx="0.002" ixy="0.0" ixz="0.0" iyy="0.002" iyz="0.0" izz="0.001"/>
             </inertial>
         </link>
@@ -39,6 +40,7 @@
             </collision>
             <inertial>
-                <mass value="1.0"/>
-                <inertia ixx="1.0" ixy="0.0" ixz="0.0" iyy="1.0" iyz="0.0" izz="1.0"/>
+                <origin xyz="0.008 0.002 -0.052"/>
+                <mass value="0.063"/>
+                <inertia ixx="0.00001" ixy="0.0" ixz="0.0" iyy="0.00001" iyz="0.0" izz="0.00001"/>
             </inertial>
         </link>
@@ -57,6 +59,7 @@
             </collision>
             <inertial>
-                <mass value="1.0"/>
-                <inertia ixx="1.0" ixy="0.0" ixz="0.0" iyy="1.0" iyz="0.0" izz="1.0"/>
+                <origin xyz="0.008 0.002 -0.052"/>
+                <mass value="0.063"/>
+                <inertia ixx="0.00001" ixy="0.0" ixz="0.0" iyy="0.00001" iyz="0.0" izz="0.00001"/>
             </inertial>
         </link>

File: src/ulixarm_description/urdf/manipulator.urdf.xacro (robot description, xacro)
@@ -22,4 +22,9 @@
                 </geometry>
             </collision>
+            <inertial>
+                <origin xyz="0. 0. 0."/>
+                <mass value="1.0"/>
+                <inertia ixx="1.0" ixy="0.0" ixz="0.0" iyy="1.0" iyz="0.0" izz="1.0"/>
+            </inertial>
         </link>
         <link name="${prefix}link1">
@@ -37,6 +42,7 @@
             </collision>
             <inertial>
-                <mass value="1.0"/>
-                <inertia ixx="1.0" ixy="0.0" ixz="0.0" iyy="1.0" iyz="0.0" izz="1.0"/>
+                <origin xyz="0. 0. 0.037"/>
+                <mass value="0.461"/>
+                <inertia ixx="0.001" ixy="0.0" ixz="0.0" iyy="0.001" iyz="0.0" izz="0.0"/>
             </inertial>
         </link>
@@ -55,6 +61,7 @@
             </collision>
             <inertial>
-                <mass value="1.0"/>
-                <inertia ixx="1.0" ixy="0.0" ixz="0.0" iyy="1.0" iyz="0.0" izz="1.0"/>
+                <origin xyz="0.197 0. -0.004"/>
+                <mass value="0.659"/>
+                <inertia ixx="0.0" ixy="0.0" ixz="0.001" iyy="0.031" iyz="0.0" izz="0.031"/>
             </inertial>
         </link>
@@ -73,6 +80,7 @@
             </collision>
             <inertial>
-                <mass value="1.0"/>
-                <inertia ixx="1.0" ixy="0.0" ixz="0.0" iyy="1.0" iyz="0.0" izz="1.0"/>
+                <origin xyz="0.197 0. -0.004"/>
+                <mass value="0.659"/>
+                <inertia ixx="0.0" ixy="0.0" ixz="0.001" iyy="0.031" iyz="0.0" izz="0.031"/>
             </inertial>
         </link>
@@ -91,6 +99,7 @@
             </collision>
             <inertial>
-                <mass value="1.0"/>
-                <inertia ixx="1.0" ixy="0.0" ixz="0.0" iyy="1.0" iyz="0.0" izz="1.0"/>
+                <origin xyz="0.022 0.0 0.018"/>
+                <mass value="0.092"/>
+                <inertia ixx="0.00001" ixy="0.0" ixz="0.0" iyy="0.00001" iyz="0.0" izz="0.00001"/>
             </inertial>
         </link>
@@ -109,12 +118,14 @@
             </collision>
             <inertial>
-                <mass value="1.0"/>
-                <inertia ixx="1.0" ixy="0.0" ixz="0.0" iyy="1.0" iyz="0.0" izz="1.0"/>
+                <origin xyz="0.030 0.0 -0.023"/>
+                <mass value="0.674"/>
+                <inertia ixx="0.001" ixy="0.0" ixz="0.0" iyy="0.002" iyz="0.0" izz="0.001"/>
             </inertial>
         </link>
         <link name="${prefix}link6">
             <inertial>
-                <mass value="1.0"/>
-                <inertia ixx="1.0" ixy="0.0" ixz="0.0" iyy="1.0" iyz="0.0" izz="1.0"/>
+                <origin xyz="0. 0. 0."/>
+                <mass value="0.001"/>
+                <inertia ixx="0.0" ixy="0.0" ixz="0.0" iyy="0.0" iyz="0.0" izz="0.00001"/>
             </inertial>
         </link>

Commit message: sync

File: src/ulixarm_description/urdf/gripper.urdf.xacro (robot description, xacro)
@@ -67,5 +67,5 @@
             <child link="${prefix}finger_right"/>
             <axis xyz="1 0 0"/>
-            <limit lower="0.0" upper="0.038" velocity="${velocity_limit_DMJ3507}" effort="${effort_limit_DMJ3507}"/>
+            <limit lower="0.0" upper="0.04" velocity="${velocity_limit_DMJ3507}" effort="${effort_limit_DMJ3507}"/>
         </joint>
         <joint name="finger_left_joint" type="prismatic">
@@ -75,5 +75,5 @@
             <axis xyz="1 0 0"/>
             <mimic joint="finger_right_joint" multiplier="1" offset="0"/>
-            <limit lower="0.0" upper="0.038" velocity="${velocity_limit_DMJ3507}" effort="${effort_limit_DMJ3507}"/>
+            <limit lower="0.0" upper="0.04" velocity="${velocity_limit_DMJ3507}" effort="${effort_limit_DMJ3507}"/>
         </joint>
   </xacro:macro>

File: src/ulixarm_moveit_config/config/ulixarm.ros2_control.xacro (robot description, xacro)
@@ -6,7 +6,10 @@
             <hardware>
                 <!-- By default, set up controllers for simulation. This won't work on real hardware -->
-                <plugin>mock_components/GenericSystem</plugin>
-                <!-- <plugin>ulixarm_hardware/RobotSystem</plugin> -->
-                <param name="port">/dev/ttyUSB0</param>
+                <!-- <plugin>mock_components/GenericSystem</plugin> -->
+                <plugin>damiao_hardware_interface/RobotSystem</plugin>
+                <param name="serial_port">/dev/ttyACM0</param>
+                <param name="serial_baud_rate">921600</param>
+                <param name="gear_pinion_module">0.001</param>
+                <param name="gear_pinion_number_teeth">14</param>
             </hardware>
             <joint name="joint1">
@@ -65,4 +68,5 @@
                 </state_interface>
                 <state_interface name="velocity"/>
+                <state_interface name="effort"/>
             </joint>
         </ros2_control>

File: src/ulixarm_moveit_config/config/ulixarm.urdf.xacro (robot description, xacro)
@@ -6,4 +6,4 @@
     <!-- Import control_xacro -->
     <xacro:include filename="ulixarm.ros2_control.xacro" />
-    <xacro:ulixarm_ros2_control name="FakeSystem" initial_positions_file="$(arg initial_positions_file)"/>
+    <xacro:ulixarm_ros2_control name="UlixarmSystem" initial_positions_file="$(arg initial_positions_file)"/>
 </robot>

Commit message: sync

File: src/ulixarm_description/urdf/gripper.urdf.xacro (robot description, xacro)
@@ -22,6 +22,7 @@
             <inertial>
                 <origin xyz="0. 0. 0.052"/>
-                <mass value="0.489"/>
-                <inertia ixx="0.002" ixy="0.0" ixz="0.0" iyy="0.002" iyz="0.0" izz="0.001"/>
+                <!-- <mass value="0.500"/> -->
+                <mass value="1.000"/>
+                <inertia ixx="0.0001" ixy="0.0" ixz="0.0" iyy="0.0001" iyz="0.0" izz="0.0001"/>
             </inertial>
         </link>
@@ -41,6 +42,6 @@
             <inertial>
                 <origin xyz="0.008 0.002 -0.052"/>
-                <mass value="0.063"/>
-                <inertia ixx="0.00001" ixy="0.0" ixz="0.0" iyy="0.00001" iyz="0.0" izz="0.00001"/>
+                <mass value="0.075"/>
+                <inertia ixx="0.0001" ixy="0.0" ixz="0.0" iyy="0.0001" iyz="0.0" izz="0.0001"/>
             </inertial>
         </link>
@@ -60,6 +61,6 @@
             <inertial>
                 <origin xyz="0.008 0.002 -0.052"/>
-                <mass value="0.063"/>
-                <inertia ixx="0.00001" ixy="0.0" ixz="0.0" iyy="0.00001" iyz="0.0" izz="0.00001"/>
+                <mass value="0.075"/>
+                <inertia ixx="0.0001" ixy="0.0" ixz="0.0" iyy="0.0001" iyz="0.0" izz="0.0001"/>
             </inertial>
         </link>

File: src/ulixarm_description/urdf/manipulator.urdf.xacro (robot description, xacro)
@@ -22,9 +22,9 @@
                 </geometry>
             </collision>
-            <inertial>
+            <!-- <inertial>
                 <origin xyz="0. 0. 0."/>
-                <mass value="1.0"/>
-                <inertia ixx="1.0" ixy="0.0" ixz="0.0" iyy="1.0" iyz="0.0" izz="1.0"/>
-            </inertial>
+                <mass value="0.0001"/>
+                <inertia ixx="0.0001" ixy="0.0" ixz="0.0" iyy="0.0001" iyz="0.0" izz="0.0001"/>
+            </inertial> -->
         </link>
         <link name="${prefix}link1">
@@ -43,6 +43,6 @@
             <inertial>
                 <origin xyz="0. 0. 0.037"/>
-                <mass value="0.461"/>
-                <inertia ixx="0.001" ixy="0.0" ixz="0.0" iyy="0.001" iyz="0.0" izz="0.0"/>
+                <mass value="0.480"/>
+                <inertia ixx="0.0001" ixy="0.0" ixz="0.0" iyy="0.0001" iyz="0.0" izz="0.0001"/>
             </inertial>
         </link>
@@ -62,6 +62,6 @@
             <inertial>
                 <origin xyz="0.197 0. -0.004"/>
-                <mass value="0.659"/>
-                <inertia ixx="0.0" ixy="0.0" ixz="0.001" iyy="0.031" iyz="0.0" izz="0.031"/>
+                <mass value="0.690"/>
+                <inertia ixx="0.0001" ixy="0.0" ixz="0.0" iyy="0.0001" iyz="0.0" izz="0.0001"/>
             </inertial>
         </link>
@@ -81,6 +81,7 @@
             <inertial>
                 <origin xyz="0.197 0. -0.004"/>
-                <mass value="0.659"/>
-                <inertia ixx="0.0" ixy="0.0" ixz="0.001" iyy="0.031" iyz="0.0" izz="0.031"/>
+                <mass value="0.680"/>
+                <!-- <mass value="0.690"/> -->
+                <inertia ixx="0.0001" ixy="0.0" ixz="0.0" iyy="0.0001" iyz="0.0" izz="0.0001"/>
             </inertial>
         </link>
@@ -100,6 +101,7 @@
             <inertial>
                 <origin xyz="0.022 0.0 0.018"/>
-                <mass value="0.092"/>
-                <inertia ixx="0.00001" ixy="0.0" ixz="0.0" iyy="0.00001" iyz="0.0" izz="0.00001"/>
+                <!-- <mass value="0.100"/> -->
+                <mass value="0.100"/>
+                <inertia ixx="0.0001" ixy="0.0" ixz="0.0" iyy="0.0001" iyz="0.0" izz="0.0001"/>
             </inertial>
         </link>
@@ -119,6 +121,7 @@
             <inertial>
                 <origin xyz="0.030 0.0 -0.023"/>
-                <mass value="0.674"/>
-                <inertia ixx="0.001" ixy="0.0" ixz="0.0" iyy="0.002" iyz="0.0" izz="0.001"/>
+                <!-- <mass value="0.700"/> -->
+                <mass value="0.700"/>
+                <inertia ixx="0.0001" ixy="0.0" ixz="0.0" iyy="0.0001" iyz="0.0" izz="0.0001"/>
             </inertial>
         </link>
@@ -127,8 +130,14 @@
                 <origin xyz="0. 0. 0."/>
                 <mass value="0.001"/>
-                <inertia ixx="0.0" ixy="0.0" ixz="0.0" iyy="0.0" iyz="0.0" izz="0.00001"/>
+                <inertia ixx="0.0001" ixy="0.0" ixz="0.0" iyy="0.0001" iyz="0.0" izz="0.0001"/>
             </inertial>
         </link>
-        <link name="${prefix}tool0"></link>
+        <link name="${prefix}tool0">
+            <inertial>
+                <origin xyz="0. 0. 0."/>
+                <mass value="0.001"/>
+                <inertia ixx="0.0001" ixy="0.0" ixz="0.0" iyy="0.0001" iyz="0.0" izz="0.0001"/>
+            </inertial>
+        </link>
         <!-- JOINTS -->
         <joint name="joint1" type="revolute">

File: src/ulixarm_description/urdf/robot.urdf (robot description, URDF)
Before this commit: robot ulixarm, 11 links, 10 joints
Links:
- link gripper_base_link: mass 1.0 -> 1.000
- link gripper_finger_left: mass 1.0 -> 0.075
- link gripper_finger_right: mass 1.0 -> 0.075
- link manipulator_link1: mass 1.0 -> 0.480
- link manipulator_link2: mass 1.0 -> 0.690
- link manipulator_link3: mass 1.0 -> 0.680
- link manipulator_link4: mass 1.0 -> 0.100
- link manipulator_link5: mass 1.0 -> 0.700
- link manipulator_link6: mass 1.0 -> 0.001
- link manipulator_tool0: mass None -> 0.001
Joints:
- joint finger_left_joint: limit lower=0.0 upper=0.038 effort=0.1 velocity=0.5 -> lower=0.0 upper=0.04 effort=0.1 velocity=0.5
- joint finger_right_joint: limit lower=0.0 upper=0.038 effort=0.1 velocity=0.5 -> lower=0.0 upper=0.04 effort=0.1 velocity=0.5

Commit message: added textures

File: src/ulixarm_description/urdf/gripper.urdf.xacro (robot description, xacro)
@@ -11,5 +11,5 @@
                 <origin xyz="0. 0. 0."/>
                 <geometry>
-                    <mesh filename="package://ulixarm_description/meshes/visual/gripper_base.stl"/>
+                    <mesh filename="package://ulixarm_description/meshes/visual/gripper_base_link.dae"/>
                 </geometry>
             </visual>
@@ -31,5 +31,5 @@
                 <origin xyz="0. 0. 0."/>
                 <geometry>
-                    <mesh filename="package://ulixarm_description/meshes/visual/finger.stl"/>
+                    <mesh filename="package://ulixarm_description/meshes/visual/finger_right.dae"/>
                 </geometry>
             </visual>

Commit message: renamed files

File: src/ulixarm_description/urdf/gripper.urdf.xacro (robot description, xacro)
@@ -17,5 +17,5 @@
                 <origin xyz="0. 0. 0."/>
                 <geometry>
-                    <mesh filename="package://ulixarm_description/meshes/collision/gripper_base.stl"/>
+                    <mesh filename="package://ulixarm_description/meshes/collision/gripper_base_link.stl"/>
                 </geometry>
             </collision>
@@ -37,5 +37,5 @@
                 <origin xyz="0. 0. 0."/>
                 <geometry>
-                    <mesh filename="package://ulixarm_description/meshes/collision/finger.stl"/>
+                    <mesh filename="package://ulixarm_description/meshes/collision/finger_right.stl"/>
                 </geometry>
             </collision>
@@ -50,5 +50,5 @@
                 <origin xyz="0. 0. 0."/>
                 <geometry>
-                    <mesh filename="package://ulixarm_description/meshes/visual/finger.stl"/>
+                    <mesh filename="package://ulixarm_description/meshes/visual/finger_right.dae"/>
                 </geometry>
             </visual>
@@ -56,5 +56,5 @@
                 <origin xyz="0. 0. 0."/>
                 <geometry>
-                    <mesh filename="package://ulixarm_description/meshes/collision/finger.stl"/>
+                    <mesh filename="package://ulixarm_description/meshes/collision/finger_right.stl"/>
                 </geometry>
             </collision>

File: src/ulixarm_description/urdf/manipulator.urdf.xacro (robot description, xacro)
@@ -19,5 +19,5 @@
                 <origin xyz="0. 0. 0."/>
                 <geometry>
-                    <mesh filename="package://ulixarm_description/meshes/collision/base.stl"/>
+                    <mesh filename="package://ulixarm_description/meshes/collision/base_link.stl"/>
                 </geometry>
             </collision>
@@ -38,5 +38,5 @@
                 <origin xyz="0. 0. 0."/>
                 <geometry>
-                    <mesh filename="package://ulixarm_description/meshes/collision/joint1.stl"/>
+                    <mesh filename="package://ulixarm_description/meshes/collision/link1.stl"/>
                 </geometry>
             </collision>
@@ -57,5 +57,5 @@
                 <origin xyz="0. 0. 0."/>
                 <geometry>
-                    <mesh filename="package://ulixarm_description/meshes/collision/link1.stl"/>
+                    <mesh filename="package://ulixarm_description/meshes/collision/link2.stl"/>
                 </geometry>
             </collision>
@@ -76,5 +76,5 @@
                 <origin xyz="0. 0. 0."/>
                 <geometry>
-                    <mesh filename="package://ulixarm_description/meshes/collision/link2.stl"/>
+                    <mesh filename="package://ulixarm_description/meshes/collision/link3.stl"/>
                 </geometry>
             </collision>
@@ -96,5 +96,5 @@
                 <origin xyz="0. 0. 0."/>
                 <geometry>
-                    <mesh filename="package://ulixarm_description/meshes/collision/joint4.stl"/>
+                    <mesh filename="package://ulixarm_description/meshes/collision/link4.stl"/>
                 </geometry>
             </collision>
@@ -116,5 +116,5 @@
                 <origin xyz="0. 0. 0."/>
                 <geometry>
-                    <mesh filename="package://ulixarm_description/meshes/collision/joint5.stl"/>
+                    <mesh filename="package://ulixarm_description/meshes/collision/link5.stl"/>
                 </geometry>
             </collision>

File: src/ulixarm_description/urdf/robot.urdf (robot description, URDF)
Before this commit: robot ulixarm, 11 links, 10 joints
Links:
- link gripper_base_link: geometry collision mesh filename=package://ulixarm_description/meshes/collision/gripper_base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; visual mesh filename=package://ulixarm_description/meshes/visual/gripper_base_li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
- link gripper_finger_left: geometry collision mesh filename=package://ulixarm_description/meshes/collision/finger_right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; visual mesh filename=package://ulixarm_description/meshes/visual/finger_right.dae
- link gripper_finger_right: geometry collision mesh filename=package://ulixarm_description/meshes/collision/finger_right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; visual mesh filename=package://ulixarm_description/meshes/visual/finger_right.dae
- link manipulator_base_link: geometry collision mesh filename=package://ulixarm_description/meshes/collision/base_link.stl; visual mesh filename=package://ulixarm_description/meshes/visual/base_link.dae
- link manipulator_link1: geometry collision mesh filename=package://ulixarm_description/meshes/collision/link1.stl; visual mesh filename=package://ulixarm_description/meshes/visual/link1.dae
- link manipulator_link2: geometry collision mesh filename=package://ulixarm_description/meshes/collision/link2.stl; visual mesh filename=package://ulixarm_description/meshes/visual/link2.dae
- link manipulator_link3: geometry collision mesh filename=package://ulixarm_description/meshes/collision/link3.stl; visual mesh filename=package://ulixarm_description/meshes/visual/link3.dae
- link manipulator_link4: geometry collision mesh filename=package://ulixarm_description/meshes/collision/link4.stl; visual mesh filename=package://ulixarm_description/meshes/visual/link4.dae
- link manipulator_link5: geometry collision mesh filename=package://ulixarm_description/meshes/collision/link5.stl; visual mesh filename=package://ulixarm_description/meshes/visual/link5.dae
