Commit message: free floating working

File: src/ulixarm_description/urdf/gripper.urdf.xacro (robot description, xacro)
@@ -22,6 +22,5 @@
             <inertial>
                 <origin xyz="0. 0. 0.052"/>
-                <!-- <mass value="0.500"/> -->
-                <mass value="1.000"/>
+                <mass value="0.450"/>
                 <inertia ixx="0.0001" ixy="0.0" ixz="0.0" iyy="0.0001" iyz="0.0" izz="0.0001"/>
             </inertial>

File: src/ulixarm_description/urdf/manipulator.urdf.xacro (robot description, xacro)
@@ -82,5 +82,4 @@
                 <origin xyz="0.197 0. -0.004"/>
                 <mass value="0.680"/>
-                <!-- <mass value="0.690"/> -->
                 <inertia ixx="0.0001" ixy="0.0" ixz="0.0" iyy="0.0001" iyz="0.0" izz="0.0001"/>
             </inertial>
@@ -101,5 +100,4 @@
             <inertial>
                 <origin xyz="0.022 0.0 0.018"/>
-                <!-- <mass value="0.100"/> -->
                 <mass value="0.100"/>
                 <inertia ixx="0.0001" ixy="0.0" ixz="0.0" iyy="0.0001" iyz="0.0" izz="0.0001"/>
@@ -121,5 +119,4 @@
             <inertial>
                 <origin xyz="0.030 0.0 -0.023"/>
-                <!-- <mass value="0.700"/> -->
                 <mass value="0.700"/>
                 <inertia ixx="0.0001" ixy="0.0" ixz="0.0" iyy="0.0001" iyz="0.0" izz="0.0001"/>

File: src/ulixarm_description/urdf/robot.urdf (robot description, URDF)
Before this commit: robot ulixarm, 11 links, 10 joints
Links:
- link gripper_base_link: mass 1.000 -> 0.450

File: src/ulixarm_moveit_config/config/ulixarm.ros2_control.xacro (robot description, xacro)
@@ -11,4 +11,5 @@
                 <param name="serial_baudrate">921600</param>
                 <param name="use_gravity_compensation">true</param> <!--true/false-->
+                <param name="use_free_floating">true</param> <!--true/false-->
             </hardware>
             <joint name="joint1">

Commit message: sync

File: src/ulixarm_description/urdf/gripper.urdf.xacro (robot description, xacro)
@@ -21,6 +21,6 @@
             </collision>
             <inertial>
-                <origin xyz="0. 0. 0.052"/>
-                <mass value="0.450"/>
+                <origin xyz="0. 0. 0.05"/>
+                <mass value="0.400"/>
                 <inertia ixx="0.0001" ixy="0.0" ixz="0.0" iyy="0.0001" iyz="0.0" izz="0.0001"/>
             </inertial>

File: src/ulixarm_description/urdf/robot.urdf (robot description, URDF)
Before this commit: robot ulixarm, 11 links, 10 joints
Links:
- link gripper_base_link: mass 0.450 -> 0.400

File: src/ulixarm_moveit_config/config/ulixarm.ros2_control.xacro (robot description, xacro)
@@ -11,8 +11,8 @@
                 <param name="serial_baudrate">921600</param>
                 <param name="use_gravity_compensation">true</param> <!--true/false-->
-                <param name="use_free_floating">true</param> <!--true/false-->
+                <param name="use_free_floating">false</param> <!--true/false-->
             </hardware>
             <joint name="joint1">
-                <param name="Kp">300.0</param>
+                <param name="Kp">20.0</param>
                 <param name="Kd">2.0</param>
                 <command_interface name="position"/>
@@ -24,6 +24,6 @@
             </joint>
             <joint name="joint2">
-                <param name="Kp">300.0</param>
-                <param name="Kd">2.0</param>
+                <param name="Kp">120.0</param>
+                <param name="Kd">3.0</param>
                 <command_interface name="position"/>
                 <command_interface name="velocity"/>
@@ -34,6 +34,6 @@
             </joint>
             <joint name="joint3">
-                <param name="Kp">300.0</param>
-                <param name="Kd">2.0</param>
+                <param name="Kp">120.0</param>
+                <param name="Kd">3.0</param>
                 <command_interface name="position"/>
                 <command_interface name="velocity"/>
@@ -44,5 +44,5 @@
             </joint>
             <joint name="joint4">
-                <param name="Kp">100.0</param>
+                <param name="Kp">10.0</param>
                 <param name="Kd">1.0</param>
                 <command_interface name="position"/>
@@ -54,5 +54,5 @@
             </joint>
             <joint name="joint5">
-                <param name="Kp">100.0</param>
+                <param name="Kp">10.0</param>
                 <param name="Kd">1.0</param>
                 <command_interface name="position"/>
@@ -65,5 +65,5 @@
             <joint name="joint6">
                 <param name="Kp">50.0</param>
-                <param name="Kd">0.5</param>
+                <param name="Kd">1.0</param>
                 <command_interface name="position"/>
                 <command_interface name="velocity"/>
@@ -74,5 +74,5 @@
             </joint>
             <joint name="finger_right_joint">
-                <param name="Kp">0.4</param>
+                <param name="Kp">0.5</param>
                 <param name="Kd">0.1</param>
                 <command_interface name="position"/>

Commit message: edit collision mesh

File: src/ulixarm_description/urdf/gripper.urdf.xacro (robot description, xacro)
@@ -66,5 +66,5 @@
         <!-- JOINTS -->
         <joint name="finger_right_joint" type="prismatic">
-            <origin xyz="0. 0. 0.1349" rpy="0. 0. 0."/>
+            <origin xyz="0. 0. 0.1289" rpy="0. 0. 0."/>
             <parent link="${prefix}base_link"/>
             <child link="${prefix}finger_right"/>
@@ -73,5 +73,5 @@
         </joint>
         <joint name="finger_left_joint" type="prismatic">
-            <origin xyz="0. 0. 0.1349" rpy="0. 0. ${PI}"/>
+            <origin xyz="0. 0. 0.1289" rpy="0. 0. ${PI}"/>
             <parent link="${prefix}base_link"/>
             <child link="${prefix}finger_left"/>

File: src/ulixarm_description/urdf/robot.urdf (robot description, URDF)
Before this commit: robot ulixarm, 11 links, 10 joints
Joints:
- joint finger_left_joint: origin xyz=0. 0. 0.1349 rpy=0. 0. 3.14159265359 -> xyz=0. 0. 0.1289 rpy=0. 0. 3.14159265359
- joint finger_right_joint: origin xyz=0. 0. 0.1349 rpy=0. 0. 0. -> xyz=0. 0. 0.1289 rpy=0. 0. 0.

File: src/ulixarm_moveit_config/config/ulixarm.ros2_control.xacro (robot description, xacro)
@@ -11,5 +11,5 @@
                 <param name="serial_baudrate">921600</param>
                 <param name="use_gravity_compensation">true</param> <!--true/false-->
-                <param name="use_free_floating">true</param> <!--true/false-->
+                <param name="use_free_floating">false</param> <!--true/false-->
             </hardware>
             <joint name="joint1">

Commit message: sync

File: src/ulixarm_description/urdf/gripper.urdf.xacro (robot description, xacro)
@@ -21,7 +21,7 @@
             </collision>
             <inertial>
-                <origin xyz="0. 0. 0.05"/>
-                <mass value="0.400"/>
-                <inertia ixx="0.0001" ixy="0.0" ixz="0.0" iyy="0.0001" iyz="0.0" izz="0.0001"/>
+                <origin xyz="0. 0. 0.052"/>
+                <mass value="0.470"/>
+                <inertia ixx="0.000337" ixy="0.0" ixz="0.0" iyy="0.000891" iyz="0.0" izz="0.000786"/>
             </inertial>
         </link>
@@ -40,7 +40,7 @@
             </collision>
             <inertial>
-                <origin xyz="0.008 0.002 -0.052"/>
-                <mass value="0.075"/>
-                <inertia ixx="0.0001" ixy="0.0" ixz="0.0" iyy="0.0001" iyz="0.0" izz="0.0001"/>
+                <origin xyz="0.010 0.002 -0.040"/>
+                <mass value="0.076"/>
+                <inertia ixx="0.000034" ixy="0.0" ixz="0.0" iyy="0.000048" iyz="0.0" izz="0.000026"/>
             </inertial>
         </link>
@@ -59,7 +59,7 @@
             </collision>
             <inertial>
-                <origin xyz="0.008 0.002 -0.052"/>
-                <mass value="0.075"/>
-                <inertia ixx="0.0001" ixy="0.0" ixz="0.0" iyy="0.0001" iyz="0.0" izz="0.0001"/>
+                <origin xyz="0.010 0.002 -0.040"/>
+                <mass value="0.076"/>
+                <inertia ixx="0.000034" ixy="0.0" ixz="0.0" iyy="0.000048" iyz="0.0" izz="0.000026"/>
             </inertial>
         </link>

File: src/ulixarm_description/urdf/manipulator.urdf.xacro (robot description, xacro)
@@ -22,9 +22,4 @@
                 </geometry>
             </collision>
-            <!-- <inertial>
-                <origin xyz="0. 0. 0."/>
-                <mass value="0.0001"/>
-                <inertia ixx="0.0001" ixy="0.0" ixz="0.0" iyy="0.0001" iyz="0.0" izz="0.0001"/>
-            </inertial> -->
         </link>
         <link name="${prefix}link1">
@@ -42,7 +37,7 @@
             </collision>
             <inertial>
-                <origin xyz="0. 0. 0.037"/>
+                <origin xyz="-0.002 0. 0.038"/>
                 <mass value="0.480"/>
-                <inertia ixx="0.0001" ixy="0.0" ixz="0.0" iyy="0.0001" iyz="0.0" izz="0.0001"/>
+                <inertia ixx="0.000288" ixy="0.0" ixz="0.0" iyy="0.000306" iyz="0.0" izz="0.000271"/>
             </inertial>
         </link>
@@ -61,7 +56,7 @@
             </collision>
             <inertial>
-                <origin xyz="0.197 0. -0.004"/>
+                <origin xyz="0.207 0. -0.003"/>
                 <mass value="0.690"/>
-                <inertia ixx="0.0001" ixy="0.0" ixz="0.0" iyy="0.0001" iyz="0.0" izz="0.0001"/>
+                <inertia ixx="0.000596" ixy="0.0" ixz="0.001074" iyy="0.009778" iyz="0.0" izz="0.009552"/>
             </inertial>
         </link>
@@ -80,7 +75,7 @@
             </collision>
             <inertial>
-                <origin xyz="0.197 0. -0.004"/>
+                <origin xyz="0.188 0. 0."/>
                 <mass value="0.680"/>
-                <inertia ixx="0.0001" ixy="0.0" ixz="0.0" iyy="0.0001" iyz="0.0" izz="0.0001"/>
+                <inertia ixx="0.000496" ixy="0.0" ixz="0.000851" iyy="0.007987" iyz="0.0" izz="0.007845"/>
             </inertial>
         </link>
@@ -99,7 +94,7 @@
             </collision>
             <inertial>
-                <origin xyz="0.022 0.0 0.018"/>
+                <origin xyz="0.022 0. 0.018"/>
                 <mass value="0.100"/>
-                <inertia ixx="0.0001" ixy="0.0" ixz="0.0" iyy="0.0001" iyz="0.0" izz="0.0001"/>
+                <inertia ixx="0.000030" ixy="0.0" ixz="0.0" iyy="0.000058" iyz="0.0" izz="0.000049"/>
             </inertial>
         </link>
@@ -118,7 +113,7 @@
             </collision>
             <inertial>
-                <origin xyz="0.030 0.0 -0.023"/>
+                <origin xyz="0.028 0. -0.024"/>
                 <mass value="0.700"/>
-                <inertia ixx="0.0001" ixy="0.0" ixz="0.0" iyy="0.0001" iyz="0.0" izz="0.0001"/>
+                <inertia ixx="0.000312" ixy="0.0" ixz="0.0" iyy="0.000892" iyz="0.0" izz="0.000911"/>
             </inertial>
         </link>
@@ -127,5 +122,5 @@
                 <origin xyz="0. 0. 0."/>
                 <mass value="0.001"/>
-                <inertia ixx="0.0001" ixy="0.0" ixz="0.0" iyy="0.0001" iyz="0.0" izz="0.0001"/>
+                <inertia ixx="0.000001" ixy="0.0" ixz="0.0" iyy="0.000001" iyz="0.0" izz="0.000001"/>
             </inertial>
         </link>
@@ -134,5 +129,5 @@
                 <origin xyz="0. 0. 0."/>
                 <mass value="0.001"/>
-                <inertia ixx="0.0001" ixy="0.0" ixz="0.0" iyy="0.0001" iyz="0.0" izz="0.0001"/>
+                <inertia ixx="0.000001" ixy="0.0" ixz="0.0" iyy="0.000001" iyz="0.0" izz="0.000001"/>
             </inertial>
         </link>
@@ -181,4 +176,5 @@
         </joint>
         <joint name="joint_tool0" type="fixed">
+            <origin xyz="0. 0. 0.1289" rpy="0. 0. 0."/>
             <parent link="${prefix}link6"/>
             <child link="${prefix}tool0"/>

File: src/ulixarm_description/urdf/robot.urdf (robot description, URDF)
Before this commit: robot ulixarm, 11 links, 10 joints
Links:
- link gripper_base_link: mass 0.400 -> 0.470
- link gripper_finger_left: mass 0.075 -> 0.076
- link gripper_finger_right: mass 0.075 -> 0.076
Joints:
- joint joint_tool0: origin (none) -> xyz=0. 0. 0.1289 rpy=0. 0. 0.
- joint manipulator_to_gripper: origin xyz=0 0 0 rpy=0 0 0 -> xyz=0 0 -0.1289 rpy=0 0 0

File: src/ulixarm_description/urdf/robot.urdf.xacro (robot description, xacro)
@@ -12,5 +12,5 @@
     <parent link="${MANIPULATOR_PREFIX}tool0"/>
     <child  link="${GRIPPER_PREFIX}base_link"/>
-    <origin xyz="0 0 0" rpy="0 0 0"/>
+    <origin xyz="0 0 -0.1289" rpy="0 0 0"/>
   </joint>
 </robot>

File: src/ulixarm_moveit_config/config/ulixarm.ros2_control.xacro (robot description, xacro)
@@ -14,6 +14,6 @@
             </hardware>
             <joint name="joint1">
-                <param name="Kp">350.0</param>
-                <param name="Kd">3.0</param>
+                <param name="Kp">500.0</param>
+                <param name="Kd">5.0</param>
                 <command_interface name="position"/>
                 <command_interface name="velocity"/>
@@ -24,6 +24,6 @@
             </joint>
             <joint name="joint2">
-                <param name="Kp">350.0</param>
-                <param name="Kd">3.0</param>
+                <param name="Kp">500.0</param>
+                <param name="Kd">5.0</param>
                 <command_interface name="position"/>
                 <command_interface name="velocity"/>
@@ -34,6 +34,6 @@
             </joint>
             <joint name="joint3">
-                <param name="Kp">300.0</param>
-                <param name="Kd">3.0</param>
+                <param name="Kp">500.0</param>
+                <param name="Kd">5.0</param>
                 <command_interface name="position"/>
                 <command_interface name="velocity"/>
@@ -44,6 +44,6 @@
             </joint>
             <joint name="joint4">
-                <param name="Kp">100.0</param>
-                <param name="Kd">1.0</param>
+                <param name="Kp">400.0</param>
+                <param name="Kd">5.0</param>
                 <command_interface name="position"/>
                 <command_interface name="velocity"/>
@@ -54,6 +54,6 @@
             </joint>
             <joint name="joint5">
-                <param name="Kp">75.0</param>
-                <param name="Kd">1.0</param>
+                <param name="Kp">300.0</param>
+                <param name="Kd">4.0</param>
                 <command_interface name="position"/>
                 <command_interface name="velocity"/>
@@ -64,6 +64,6 @@
             </joint>
             <joint name="joint6">
-                <param name="Kp">50.0</param>
-                <param name="Kd">1.0</param>
+                <param name="Kp">100.0</param>
+                <param name="Kd">3.0</param>
                 <command_interface name="position"/>
                 <command_interface name="velocity"/>
