Commit message: added visuals

File: src/ulixarm_description/urdf/gripper.urdf.xacro (robot description, xacro)
@@ -4,6 +4,4 @@
         <!-- CONSTANTS -->
         <xacro:property name="PI" value="3.14159265359"/>
-        <xacro:property name="velocity_limit_DMJ3507"   value="0.5"/>
-        <xacro:property name="effort_limit_DMJ3507"     value="0.1"/>
         <!-- LINKS -->
         <link name="${prefix}base_link">
@@ -11,5 +9,5 @@
                 <origin xyz="0. 0. 0."/>
                 <geometry>
-                    <mesh filename="package://ulixarm_description/meshes/visual/gripper_base_link.dae"/>
+                    <mesh filename="package://ulixarm_description/meshes/visual/gripper.dae"/>
                 </geometry>
             </visual>
@@ -21,7 +19,7 @@
             </collision>
             <inertial>
-                <origin xyz="0. 0. 0.052"/>
-                <mass value="0.470"/>
-                <inertia ixx="0.000337" ixy="0.0" ixz="0.0" iyy="0.000891" iyz="0.0" izz="0.000786"/>
+                <origin xyz="-0.012 0. 0.036"/>
+                <mass value="0.730"/>
+                <inertia ixx="0.000939" ixy="0.0" ixz="0.0" iyy="0.000987" iyz="0.0" izz="0.001086"/>
             </inertial>
         </link>
@@ -30,5 +28,5 @@
                 <origin xyz="0. 0. 0."/>
                 <geometry>
-                    <mesh filename="package://ulixarm_description/meshes/visual/finger_right.dae"/>
+                    <mesh filename="package://ulixarm_description/meshes/visual/finger.dae"/>
                 </geometry>
             </visual>
@@ -49,5 +47,5 @@
                 <origin xyz="0. 0. 0."/>
                 <geometry>
-                    <mesh filename="package://ulixarm_description/meshes/visual/finger_right.dae"/>
+                    <mesh filename="package://ulixarm_description/meshes/visual/finger.dae"/>
                 </geometry>
             </visual>
@@ -66,17 +64,17 @@
         <!-- JOINTS -->
         <joint name="finger_right_joint" type="prismatic">
-            <origin xyz="0. 0. 0.1289" rpy="0. 0. 0."/>
+            <origin xyz="0. 0. 0.0745" rpy="0. 0. ${PI/2}"/>
             <parent link="${prefix}base_link"/>
             <child link="${prefix}finger_right"/>
             <axis xyz="1 0 0"/>
-            <limit lower="0.0" upper="0.04" velocity="${velocity_limit_DMJ3507}" effort="${effort_limit_DMJ3507}"/>
+            <limit lower="0.0" upper="0.045" velocity="0.0" effort="0.0"/>
         </joint>
         <joint name="finger_left_joint" type="prismatic">
-            <origin xyz="0. 0. 0.1289" rpy="0. 0. ${PI}"/>
+            <origin xyz="0. 0. 0.0745" rpy="0. 0. ${-PI/2}"/>
             <parent link="${prefix}base_link"/>
             <child link="${prefix}finger_left"/>
             <axis xyz="1 0 0"/>
             <mimic joint="finger_right_joint" multiplier="1" offset="0"/>
-            <limit lower="0.0" upper="0.04" velocity="${velocity_limit_DMJ3507}" effort="${effort_limit_DMJ3507}"/>
+            <limit lower="0.0" upper="0.045" velocity="0.0" effort="0.0"/>
         </joint>
   </xacro:macro>

File: src/ulixarm_description/urdf/manipulator.urdf.xacro (robot description, xacro)
@@ -37,7 +37,7 @@
             </collision>
             <inertial>
-                <origin xyz="-0.002 0. 0.038"/>
-                <mass value="0.480"/>
-                <inertia ixx="0.000288" ixy="0.0" ixz="0.0" iyy="0.000306" iyz="0.0" izz="0.000271"/>
+                <origin xyz="0. 0.002 0.043"/>
+                <mass value="0.575"/>
+                <inertia ixx="0.000434" ixy="0.0" ixz="0.0" iyy="0.000387" iyz="0.0" izz="0.000326"/>
             </inertial>
         </link>
@@ -56,7 +56,7 @@
             </collision>
             <inertial>
-                <origin xyz="0.207 0. -0.003"/>
-                <mass value="0.690"/>
-                <inertia ixx="0.000596" ixy="0.0" ixz="0.001074" iyy="0.009778" iyz="0.0" izz="0.009552"/>
+                <origin xyz="0.207 0. -0.005"/>
+                <mass value="0.887"/>
+                <inertia ixx="0.000679" ixy="0.0" ixz="0.001200" iyy="0.010762" iyz="0.0" izz="0.010534"/>
             </inertial>
         </link>
@@ -75,7 +75,7 @@
             </collision>
             <inertial>
-                <origin xyz="0.188 0. 0."/>
-                <mass value="0.680"/>
-                <inertia ixx="0.000496" ixy="0.0" ixz="0.000851" iyy="0.007987" iyz="0.0" izz="0.007845"/>
+                <origin xyz="0.202 0. -0.004"/>
+                <mass value="0.819"/>
+                <inertia ixx="0.000572" ixy="0.0" ixz="0.001045" iyy="0.010133" iyz="0.0" izz="0.009994"/>
             </inertial>
         </link>
@@ -94,7 +94,7 @@
             </collision>
             <inertial>
-                <origin xyz="0.022 0. 0.018"/>
-                <mass value="0.100"/>
-                <inertia ixx="0.000030" ixy="0.0" ixz="0.0" iyy="0.000058" iyz="0.0" izz="0.000049"/>
+                <origin xyz="0.024 -0.017 0.048"/>
+                <mass value="0.072"/>
+                <inertia ixx="0.000075" ixy="0.0" ixz="0.0" iyy="0.000084" iyz="0.0" izz="0.000095"/>
             </inertial>
         </link>
@@ -113,13 +113,25 @@
             </collision>
             <inertial>
-                <origin xyz="0.028 0. -0.024"/>
-                <mass value="0.700"/>
-                <inertia ixx="0.000312" ixy="0.0" ixz="0.0" iyy="0.000892" iyz="0.0" izz="0.000911"/>
+                <origin xyz="0.028 0. -0.027"/>
+                <mass value="0.786"/>
+                <inertia ixx="0.000379" ixy="0.0" ixz="0.0" iyy="0.001085" iyz="0.0" izz="0.001097"/>
             </inertial>
         </link>
         <link name="${prefix}link6">
+            <visual>
+                <origin xyz="0. 0. 0."/>
+                <geometry>
+                    <mesh filename="package://ulixarm_description/meshes/visual/link6.dae"/>
+                </geometry>
+            </visual>
+            <collision>
+                <origin xyz="0. 0. 0."/>
+                <geometry>
+                    <mesh filename="package://ulixarm_description/meshes/collision/link5.stl"/>
+                </geometry>
+            </collision>
             <inertial>
-                <origin xyz="0. 0. 0."/>
-                <mass value="0.001"/>
+                <origin xyz="0. 0. 0.007"/>
+                <mass value="0.025"/>
                 <inertia ixx="0.000001" ixy="0.0" ixz="0.0" iyy="0.000001" iyz="0.0" izz="0.000001"/>
             </inertial>
@@ -129,52 +141,52 @@
                 <origin xyz="0. 0. 0."/>
                 <mass value="0.001"/>
-                <inertia ixx="0.000001" ixy="0.0" ixz="0.0" iyy="0.000001" iyz="0.0" izz="0.000001"/>
+                <inertia ixx="0.000004" ixy="0.0" ixz="0.0" iyy="0.000003" iyz="0.0" izz="0.000006"/>
             </inertial>
         </link>
         <!-- JOINTS -->
         <joint name="joint1" type="revolute">
-            <origin xyz="0. 0. 0.0533" rpy="0. 0. 0."/>
+            <origin xyz="0. 0. 0.0645" rpy="0. 0. 0."/>
             <parent link="${prefix}base_link"/>
             <child link="${prefix}link1"/>
             <axis xyz="0 0 1"/>
-            <limit lower="${-PI/2}" upper="${PI/2}" velocity="${velocity_limit_DM4340}" effort="${effort_limit_DM4340}"/>
+            <limit lower="-1.8326" upper="1.8326" velocity="${velocity_limit_DM4340}" effort="${effort_limit_DM4340}"/>
         </joint>
         <joint name="joint2" type="revolute">
-            <origin xyz="0.027175 0. 0.0425" rpy="${PI} ${-PI/2} 0."/>
+            <origin xyz="0. -0.031175 0.0495" rpy="${PI/2} ${-PI/2} 0."/>
             <parent link="${prefix}link1"/>
             <child link="${prefix}link2"/>
             <axis xyz="0 0 1"/>
-            <limit lower="${-PI/2}" upper="${PI/2}" velocity="${velocity_limit_DM4340}" effort="${effort_limit_DM4340}"/>
+            <limit lower="${-PI/2}" upper="1.25664" velocity="${velocity_limit_DM4340}" effort="${effort_limit_DM4340}"/>
         </joint>
         <joint name="joint3" type="revolute">
-            <origin xyz="0.280 0. -0.0473" rpy="${PI} 0. 0."/>
+            <origin xyz="0.280 0. -0.0523" rpy="0. ${PI} ${PI}"/>
             <parent link="${prefix}link2"/>
             <child link="${prefix}link3"/>
             <axis xyz="0 0 1"/>
-            <limit lower="${-PI/2}" upper="2.7925268" velocity="${velocity_limit_DM4340}" effort="${effort_limit_DM4340}"/>
+            <limit lower="${-PI/2}" upper="2.82743" velocity="${velocity_limit_DM4340}" effort="${effort_limit_DM4340}"/>
         </joint>
         <joint name="joint4" type="revolute">
-            <origin xyz="0.260 0. -0.040" rpy="${PI} 0. ${-PI/2}"/>
+            <origin xyz="0.280 0. -0.046" rpy="0. ${PI} ${PI}"/>
             <parent link="${prefix}link3"/>
             <child link="${prefix}link4"/>
             <axis xyz="0 0 1"/>
-            <limit lower="${-PI}" upper="${PI/2}" velocity="${velocity_limit_DM4310}" effort="${effort_limit_DM4310}"/>
+            <limit lower="${-PI/2}" upper="2.61799" velocity="${velocity_limit_DM4310}" effort="${effort_limit_DM4310}"/>
         </joint>
         <joint name="joint5" type="revolute">
-            <origin xyz="0.046 0. 0.031" rpy="${PI/2} 0. ${-PI/2}"/>
+            <origin xyz="0.052 -0.036 -0.034" rpy="${PI/2} 0. ${-PI/2}"/>
             <parent link="${prefix}link4"/>
             <child link="${prefix}link5"/>
             <axis xyz="0 0 -1"/>
-            <limit lower="${-PI/2}" upper="${PI/2}" velocity="${velocity_limit_DM4310}" effort="${effort_limit_DM4310}"/>
+            <limit lower="-1.8326" upper="1.8326" velocity="${velocity_limit_DM4310}" effort="${effort_limit_DM4310}"/>
         </joint>
         <joint name="joint6" type="revolute">
-            <origin xyz="0.0825 0. -0.0235" rpy="${PI/2} 0. ${PI/2}"/>
+            <origin xyz="0.0855 0. -0.0265" rpy="${PI} ${-PI/2} 0."/>
             <parent link="${prefix}link5"/>
             <child link="${prefix}link6"/>
             <axis xyz="0 0 1"/>
-            <limit lower="${-PI/2}" upper="${PI/2}" velocity="${velocity_limit_DM4310}" effort="${effort_limit_DM4310}"/>
+            <limit lower="-2.93215" upper="2.93215" velocity="${velocity_limit_DM4310}" effort="${effort_limit_DM4310}"/>
         </joint>
         <joint name="joint_tool0" type="fixed">
-            <origin xyz="0. 0. 0.1289" rpy="0. 0. 0."/>
+            <origin xyz="0. 0. 0.005" rpy="0. 0. 0."/>
             <parent link="${prefix}link6"/>
             <child link="${prefix}tool0"/>

File: src/ulixarm_description/urdf/robot.urdf (robot description, URDF)
Before this commit: robot ulixarm, 11 links, 10 joints
Links:
- link gripper_base_link: mass 0.470 -> 0.730; geometry collision mesh filename=package://ulixarm_description/meshes/collision/gripper_base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; visual mesh filename=package://ulixarm_description/meshes/visual/gripper.dae
- link gripper_finger_left: geometry collision mesh filename=package://ulixarm_description/meshes/collision/finger_right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; visual mesh filename=package://ulixarm_description/meshes/visual/finger.dae
- link gripper_finger_right: geometry collision mesh filename=package://ulixarm_description/meshes/collision/finger_right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; visual mesh filename=package://ulixarm_description/meshes/visual/finger.dae
- link manipulator_link1: mass 0.480 -> 0.575
- link manipulator_link2: mass 0.690 -> 0.887
- link manipulator_link3: mass 0.680 -> 0.819
- link manipulator_link4: mass 0.100 -> 0.072
- link manipulator_link5: mass 0.700 -> 0.786
- link manipulator_link6: mass 0.001 -> 0.025; geometry collision mesh filename=package://ulixarm_description/meshes/collision/link5.stl; visual mesh filename=package://ulixarm_description/meshes/visual/link6.dae
Joints:
- joint finger_left_joint: limit lower=0.0 upper=0.04 effort=0.1 velocity=0.5 -> lower=0.0 upper=0.045 effort=0.0 velocity=0.0; origin xyz=0. 0. 0.1289 rpy=0. 0. 3.14159265359 -> xyz=0. 0. 0.0745 rpy=0. 0. -1.570796326795
- joint finger_right_joint: limit lower=0.0 upper=0.04 effort=0.1 velocity=0.5 -> lower=0.0 upper=0.045 effort=0.0 velocity=0.0; origin xyz=0. 0. 0.1289 rpy=0. 0. 0. -> xyz=0. 0. 0.0745 rpy=0. 0. 1.570796326795
- joint joint1: limit lower=-1.570796326795 upper=1.570796326795 effort=27.0 velocity=8.0 -> lower=-1.8326 upper=1.8326 effort=27.0 velocity=8.0; origin xyz=0. 0. 0.0533 rpy=0. 0. 0. -> xyz=0. 0. 0.0645 rpy=0. 0. 0.
- joint joint2: limit lower=-1.570796326795 upper=1.570796326795 effort=27.0 velocity=8.0 -> lower=-1.570796326795 upper=1.25664 effort=27.0 velocity=8.0; origin xyz=0.027175 0. 0.0425 rpy=3.14159265359 -1.570796326795 0. -> xyz=0. -0.031175 0.0495 rpy=1.570796326795 -1.570796326795 0.
- joint joint3: limit lower=-1.570796326795 upper=2.7925268 effort=27.0 velocity=8.0 -> lower=-1.570796326795 upper=2.82743 effort=27.0 velocity=8.0; origin xyz=0.280 0. -0.0473 rpy=3.14159265359 0. 0. -> xyz=0.280 0. -0.0523 rpy=0. 3.14159265359 3.14159265359
- joint joint4: limit lower=-3.14159265359 upper=1.570796326795 effort=10.0 velocity=30.0 -> lower=-1.570796326795 upper=2.61799 effort=10.0 velocity=30.0; origin xyz=0.260 0. -0.040 rpy=3.14159265359 0. -1.570796326795 -> xyz=0.280 0. -0.046 rpy=0. 3.14159265359 3.14159265359
- joint joint5: limit lower=-1.570796326795 upper=1.570796326795 effort=10.0 velocity=30.0 -> lower=-1.8326 upper=1.8326 effort=10.0 velocity=30.0; origin xyz=0.046 0. 0.031 rpy=1.570796326795 0. -1.570796326795 -> xyz=0.052 -0.036 -0.034 rpy=1.570796326795 0. -1.570796326795
- joint joint6: limit lower=-1.570796326795 upper=1.570796326795 effort=10.0 velocity=30.0 -> lower=-2.93215 upper=2.93215 effort=10.0 velocity=30.0; origin xyz=0.0825 0. -0.0235 rpy=1.570796326795 0. 1.570796326795 -> xyz=0.0855 0. -0.0265 rpy=3.14159265359 -1.570796326795 0.
- joint joint_tool0: origin xyz=0. 0. 0.1289 rpy=0. 0. 0. -> xyz=0. 0. 0.005 rpy=0. 0. 0.
- joint manipulator_to_gripper: origin xyz=0 0 -0.1289 rpy=0 0 0 -> xyz=0 0 0 rpy=0 0 0

File: src/ulixarm_description/urdf/robot.urdf.xacro (robot description, xacro)
@@ -12,5 +12,5 @@
     <parent link="${MANIPULATOR_PREFIX}tool0"/>
     <child  link="${GRIPPER_PREFIX}base_link"/>
-    <origin xyz="0 0 -0.1289" rpy="0 0 0"/>
+    <origin xyz="0 0 0" rpy="0 0 0"/>
   </joint>
 </robot>

Commit message: added collision

File: src/ulixarm_description/urdf/gripper.urdf.xacro (robot description, xacro)
@@ -15,5 +15,5 @@
                 <origin xyz="0. 0. 0."/>
                 <geometry>
-                    <mesh filename="package://ulixarm_description/meshes/collision/gripper_base_link.stl"/>
+                    <mesh filename="package://ulixarm_description/meshes/collision/gripper.stl"/>
                 </geometry>
             </collision>
@@ -34,5 +34,5 @@
                 <origin xyz="0. 0. 0."/>
                 <geometry>
-                    <mesh filename="package://ulixarm_description/meshes/collision/finger_right.stl"/>
+                    <mesh filename="package://ulixarm_description/meshes/collision/finger.stl"/>
                 </geometry>
             </collision>
@@ -53,5 +53,5 @@
                 <origin xyz="0. 0. 0."/>
                 <geometry>
-                    <mesh filename="package://ulixarm_description/meshes/collision/finger_right.stl"/>
+                    <mesh filename="package://ulixarm_description/meshes/collision/finger.stl"/>
                 </geometry>
             </collision>
@@ -68,5 +68,5 @@
             <child link="${prefix}finger_right"/>
             <axis xyz="1 0 0"/>
-            <limit lower="0.0" upper="0.045" velocity="0.0" effort="0.0"/>
+            <limit lower="0.0" upper="0.045" velocity="0.5" effort="10.0"/>
         </joint>
         <joint name="finger_left_joint" type="prismatic">
@@ -76,5 +76,5 @@
             <axis xyz="1 0 0"/>
             <mimic joint="finger_right_joint" multiplier="1" offset="0"/>
-            <limit lower="0.0" upper="0.045" velocity="0.0" effort="0.0"/>
+            <limit lower="0.0" upper="0.045" velocity="0.5" effort="10.0"/>
         </joint>
   </xacro:macro>

File: src/ulixarm_description/urdf/manipulator.urdf.xacro (robot description, xacro)
@@ -125,10 +125,4 @@
                 </geometry>
             </visual>
-            <collision>
-                <origin xyz="0. 0. 0."/>
-                <geometry>
-                    <mesh filename="package://ulixarm_description/meshes/collision/link5.stl"/>
-                </geometry>
-            </collision>
             <inertial>
                 <origin xyz="0. 0. 0.007"/>

File: src/ulixarm_description/urdf/robot.urdf (robot description, URDF)
Before this commit: robot ulixarm, 11 links, 10 joints
Links:
- link gripper_base_link: geometry collision mesh filename=package://ulixarm_description/meshes/collision/gripper.stl; visual mesh filename=package://ulixarm_description/meshes/visual/gripper.dae
- link gripper_finger_left: geometry collision mesh filename=package://ulixarm_description/meshes/collision/finger.stl; visual mesh filename=package://ulixarm_description/meshes/visual/finger.dae
- link gripper_finger_right: geometry collision mesh filename=package://ulixarm_description/meshes/collision/finger.stl; visual mesh filename=package://ulixarm_description/meshes/visual/finger.dae
- link manipulator_link6: geometry visual mesh filename=package://ulixarm_description/meshes/visual/link6.dae
Joints:
- joint finger_left_joint: limit lower=0.0 upper=0.045 effort=0.0 velocity=0.0 -> lower=0.0 upper=0.045 effort=10.0 velocity=0.5
- joint finger_right_joint: limit lower=0.0 upper=0.045 effort=0.0 velocity=0.0 -> lower=0.0 upper=0.045 effort=10.0 velocity=0.5

Commit message: edit gripper mass

File: src/ulixarm_description/urdf/gripper.urdf.xacro (robot description, xacro)
@@ -20,5 +20,5 @@
             <inertial>
                 <origin xyz="-0.012 0. 0.036"/>
-                <mass value="0.730"/>
+                <mass value="0.73"/>
                 <inertia ixx="0.000939" ixy="0.0" ixz="0.0" iyy="0.000987" iyz="0.0" izz="0.001086"/>
             </inertial>
@@ -39,5 +39,5 @@
             <inertial>
                 <origin xyz="0.010 0.002 -0.040"/>
-                <mass value="0.076"/>
+                <mass value="0.0"/>
                 <inertia ixx="0.000034" ixy="0.0" ixz="0.0" iyy="0.000048" iyz="0.0" izz="0.000026"/>
             </inertial>
@@ -58,5 +58,5 @@
             <inertial>
                 <origin xyz="0.010 0.002 -0.040"/>
-                <mass value="0.076"/>
+                <mass value="0.0"/>
                 <inertia ixx="0.000034" ixy="0.0" ixz="0.0" iyy="0.000048" iyz="0.0" izz="0.000026"/>
             </inertial>

File: src/ulixarm_description/urdf/robot.urdf (robot description, URDF)
Before this commit: robot ulixarm, 11 links, 10 joints
Links:
- link gripper_base_link: mass 0.730 -> 0.73
- link gripper_finger_left: mass 0.076 -> 0.0
- link gripper_finger_right: mass 0.076 -> 0.0
